File: KICAD/SSR-PCB/SSR-PCB.kicad_pcb (KiCad board)
At the start: 4 copper layers, 80 x 75 mm, 8 parts, among them J1 Conn_01x02, J2 Screw_Terminal_01x02

Commit message: KiCAD edits
Parts:
- moved J2 3.81 mm to (-140.0, 27.5), turned to 180 degrees
Routing:
- net Net-(J2-Pad2): track 17.2 -> 44.8 mm
- net Net-(J2-Pad1): track 17.2 -> 22.2 mm
- net GND: track 23.0 -> 24.2 mm
