File: KICAD/base8x/base8x.kicad_pcb (KiCad board)
At the start: 4 copper layers, 210 x 130 mm, 35 parts, among them J1 Conn_02x05_Odd_Even, J2 GS3, J3 Conn_02x14_Counter_Clockwise, J4 GS3, J5 Conn_01x02, J9 Screw_Terminal_01x08, P3 CONN_01X02, P4 CONN_01X02, U1 ADS1115

Commit message: Chanign track sizes and re producing drill files
Parts:
- moved Raspberry_header1 5.33 mm to (-217.8, 53.7)
Routing:
- net SDA: track 174.9 -> 125.2 mm, vias 5 -> 7
- net A_V_D_EXT: track 172.8 -> 203.1 mm
- net MOSI: track 162.7 -> 183.1 mm, vias 3 -> 5
- net +5V: track 31.1 -> 48.4 mm, vias 6 -> 7
- net MISO: track 143.3 -> 150.2 mm, vias 4 -> 3
- net SCL: track 164.5 -> 170.9 mm, vias 4 -> 6
- net +3V3: track 91.8 -> 97.3 mm
- net GPIO6: track 28.7 -> 23.9 mm
- net SCK: track 75.9 -> 79.3 mm
- net CLK0: track 123.5 -> 125.2 mm
- net A_V_D: track 60.1 -> 61.7 mm

Commit message: Changing Via sizes and track widths
Parts:
- removed REF** (x4): MountingHole_3.2mm_M3, MountingHole:MountingHole_3.2mm_M3
- removed U1: ADS1115, Package_SO:MSOP-10_3x3mm_P0.5mm
- added IC1: ADS1115, base8x:ADS1115, F.Cu at (-282.4, 110.0)
- moved TP2 62.3 mm to (-305.6, 100.1)
- moved C1 60.2 mm to (-271.8, 110.0)
Connections:
- J3 pad 12: Net-(J3-Pad12) -> ~A_CS
- J3 pad 16: A_V_D -> Net-(J3-Pad16)
- J4 pad 1: +5V -> GND
- J4 pad 3: GND -> +5V
- R4 pad 1: Net-(J4-Pad2) -> Net-(IC1-Pad5)
- R4 pad 2: Net-(R4-Pad2) -> Net-(J4-Pad2)
Routing:
- net ~A_CS: track 71.7 -> 186.6 mm, vias 4 -> 2
- net GND: track 90.8 -> 170.7 mm, vias 8 -> 4
- net SCL: track 170.9 -> 243.3 mm, vias 6 -> 8
- net SDA: track 125.2 -> 180.9 mm, vias 7 -> 6
- net Net-(IC1-Pad9): track 108.3 -> 163.4 mm
- net Net-(R4-Pad2): track 53.5 -> 0.00 mm, vias 1 -> 0
- net Net-(IC1-Pad5): track 0.00 -> 50.7 mm, vias 0 -> 2
- net A_V_D_LOC: track 25.5 -> 66.7 mm
- net A_V_D: track 61.7 -> 41.1 mm
- net +5V: track 48.4 -> 66.4 mm, vias 7 -> 6
- net Net-(IC1-Pad6): track 29.4 -> 46.1 mm, vias 0 -> 2
- net SCK: track 79.3 -> 94.6 mm, vias 3 -> 2
- net MOSI: track 183.1 -> 194.4 mm
- net A_V_D_EXT: track 203.1 -> 192.0 mm, vias 2 -> 1
- net Net-(J4-Pad2): track 46.2 -> 36.4 mm
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Other:
- net class Default: clearance 0.16 -> 0.3; trace_width 0.25 -> 1; via_dia 0.6 -> 1; via_drill 0.4 -> 0.8
- rule trace_clearance: 0.16 -> 0.3
- rule trace_min: 0.25 -> 0.9
- rule via_min_size: 0.4 -> 0.8
