File: KICAD/base8x/base8x.sch (KiCad schematic (older format))
At the start: 31 parts, among them J1 Conn_02x05_Odd_Even, J2 GS3, J3 Conn_02x14_Counter_Clockwise, J4 GS3, J5 Conn_01x02, J9 Screw_Terminal_01x08, P3 CONN_01X02, P4 CONN_01X02, U1 ADS1115

Commit message: Changing Via sizes and track widths
Parts:
- removed U1: ADS1115, Package_SO:MSOP-10_3x3mm_P0.5mm, symbol base8x-rescue:ADS1115-myParts
- added IC1: ADS1115, base8x:ADS1115, symbol ADS1115:ADS1115
Connections:
- wire segments 86 -> 94
- no-connect marks 40 -> 42
Other:
- moved on the sheet: C1, D1, D2, J4, JP2, JP3, JP4, JP5, R1, R2, R3, R4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
